File: pico/kicad/pico-brook-.kicad_pcb (KiCad board)
At the start: 2 copper layers, 96.2 x 45.2 mm, 16 parts, among them J10 Conn_01x03_Male, J11 Conn_01x04_Female, J2 Conn_01x05_Male, J3 Screw_Terminal_01x20, J4 Conn_01x04_Male, J5 Conn_01x05_Male, J6 Conn_01x04_Male, J7 Conn_01x04_Male, J8 Conn_01x04_Male, J9 Conn_02x10_Odd_Even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

Commit message: Minor adjustments to traces, remove J2 and J5 due to nonuse
Parts:
- removed J2, J5: Conn_01x05_Male, Connector_PinHeader_2.00mm:PinHeader_1x05_P2.00mm_Vertical
- removed REF**: PinHeader_1x02_P2.54mm_Vertical, Connector_PinHeader_2.54mm:PinHeader_1x02_P2.54mm_Vertical
Routing:
- net TURBO: track 72.9 -> 67.0 mm
- net TURBO LED: track 66.2 -> 60.3 mm
